File: PCB/OpenThereminV4.kicad_pcb (KiCad board)
At the start: 2 copper layers, 50.5 x 128.5 mm, 105 parts, among them J1 USB_C_Receptacle, J2 Conn_02x03_Odd_Even, P1 10k, P10 BUTTON, P11 A3_PAD, P12 A2_PAD, P13 A1_PAD, P14 A0_PAD, P2 10k, P3 10k, P4 10k, P8 VCC, P9 GND, U1 TTP223, U10 CH340G, U11 LP2985-3.3, U12 MCP4922-E/SL, U2 4060, U3 4060, U4 74HC74, U5 4069, U6 MCP4921-E/SN, U7 MCP4922-E/SL, U8 LM358 / MCP6002, U9 ATmega328P-AU, X1 16MHz, X2 7.3721MHz, X3 12MHz, Y1 MountPad3, Y2 MountPad3, Y3 PLUG_3_5_SMD, Y7 PLUG_3_5_SMD

Commit message: Finalized Prototype design will test soon
Parts:
- added P15: CV2, GaudiLabsFootPrints:SMD_Pinheader_1_OT_BLANK, B.Cu at (122.5, 154.9)
- added P16: GND, GaudiLabsFootPrints:SMD_Pinheader_1_OT_BLANK, B.Cu at (122.5, 138.4)
- added P5: VCC, GaudiLabsFootPrints:SMD_Pinheader_1_OT_BLANK, B.Cu at (122.5, 108.4)
- added P6: audio, GaudiLabsFootPrints:SMD_Pinheader_1_OT_BLANK, B.Cu at (122.5, 141.0)
- added P7: CV1, GaudiLabsFootPrints:SMD_Pinheader_1_OT_BLANK, B.Cu at (122.5, 152.4)
- W1, W2: footprint Fiducials:Fiducial_1mm_Dia_2.54mm_Outer_CopperTop -> GaudiLabsFootPrints:Fiducial_1mm_Dia_2.54mm_Outer_CopperBottom; moved to B.Cu
- moved W1 59.1 mm to (122.0, 70.0)
- moved W2 51.5 mm to (78.0, 155.0)
- moved C37 0.43 mm to (121.2, 110.7)
Routing:
- net Net-(P15-Pad1): track 13.2 -> 27.9 mm
- net Net-(P7-Pad1): track 29.2 -> 42.2 mm
- net RXD: track 26.7 -> 34.8 mm, vias 2 -> 4
- net GND: track 119.7 -> 127.3 mm, vias 33 -> 35
- net Net-(C29-Pad2): track 9.20 -> 16.5 mm
- net EX_CLK: track 38.5 -> 40.6 mm
- net VCC: track 309.0 -> 309.6 mm
Other:
- board size 50.5 x 128.5 mm -> 50.5 x 127.5 mm
- board text added: "AUDIO"
- board text added: "CV1"
- board text added: "CV2"
- board text added: "GD"
- board text added: "TX"
