File: PCB/OpenThereminV4.sch (KiCad schematic (older format))
At the start: 101 parts, among them J1 USB_C_Receptacle, J2 Conn_02x03_Odd_Even, P1 10k, P10 BUTTON, P11 A3_PAD, P12 A2_PAD, P13 A1_PAD, P14 A0_PAD, P2 10k, P3 10k, P4 10k, P8 VCC, P9 GND, U1 TTP223, U10 CH340G, U11 LP2985-3.3, U12 MCP4922-E/SL, U2 4060, U3 4060, U4 74HC74, U5 4069, U6 MCP4921-E/SN, U7 MCP4922-E/SL, U8 LM358 / MCP6002, U9 ATmega328P-AU, X1 16MHz, X2 7.3721MHz, X3 12MHz, Y1 MountPad3, Y2 MountPad3, Y3 PLUG_3_5_SMD, Y7 PLUG_3_5_SMD

Commit message: Finalized Prototype design will test soon
Parts:
- removed W3: TP1, Measurement_Points:Measurement_Point_Round-SMD-Pad_Small, symbol OpenThereminV4-rescue:TEST_1P
- removed W4: TP2, Measurement_Points:Measurement_Point_Round-SMD-Pad_Small, symbol OpenThereminV4-rescue:TEST_1P
- added P15: CV2, GaudiLabsFootPrints:SMD_Pinheader_1_OT_BLANK, symbol OpenThereminV4-rescue:CONN_01X01
- added P16: GND, GaudiLabsFootPrints:SMD_Pinheader_1_OT_BLANK, symbol OpenThereminV4-rescue:CONN_01X01
- added P5: VCC, GaudiLabsFootPrints:SMD_Pinheader_1_OT_BLANK, symbol OpenThereminV4-rescue:CONN_01X01
- added P6: audio, GaudiLabsFootPrints:SMD_Pinheader_1_OT_BLANK, symbol OpenThereminV4-rescue:CONN_01X01
- added P7: CV1, GaudiLabsFootPrints:SMD_Pinheader_1_OT_BLANK, symbol OpenThereminV4-rescue:CONN_01X01
- W1, W2: footprint Fiducials:Fiducial_1mm_Dia_2.54mm_Outer_CopperTop -> GaudiLabsFootPrints:Fiducial_1mm_Dia_2.54mm_Outer_CopperBottom
Connections:
- net GND: now also P16.1 (P1)
- net RXD: now also P5.1 (P1)
- net at C29.2, Y7.3 (L): now also P6.1 (P1)
- net at U12.10 (VoutB), Y3.2 (R): now also P15.1 (P1)
- net at U12.14 (VoutA), Y3.3 (L): now also P7.1 (P1)
Changed lines of the file:
@@
 	1    0    0    -1
 $EndComp
-Text Notes 9650 1950 0    60   ~ 0
+Text Notes 11450 1350 0    60   ~ 0
 MCP 6402-E/SN
-Text Notes 9700 2050 0    60   ~ 0
+Text Notes 11450 1450 0    60   ~ 0
 MCP60x\n
-Text Notes 9750 2150 0    60   ~ 0
+Text Notes 11450 1550 0    60   ~ 0
 LMV358M8G-13\n
 $Comp
@@
 	6000 2850 5900 2850
 Wire Wire Line
-	5900 2850 5900 1850
-Wire Wire Line
 	3650 5250 3750 5250
 Wire Wire Line
@@
 $EndComp
 Wire Wire Line
-	10700 1550 10700 2000
+	10700 1550 10700 1650
 $Comp
 L OpenThereminV4-rescue:GND #PWR038
@@
 Wire Wire Line
 	10200 1550 10350 1550
-Text Label 10900 2050 0    60   ~ 0
+Text Label 11500 1850 0    60   ~ 0
 JMP
 $Comp
@@
 F 0 "W1" V 5800 7650 50  0000 C CNN
 F 1 "FIDUCIAL1" V 5900 8000 50  0000 C CNN
-F 2 "Fiducials:Fiducial_1mm_Dia_2.54mm_Outer_CopperTop" H 6100 7600 50  0001 C CNN
+F 2 "GaudiLabsFootPrints:Fiducial_1mm_Dia_2.54mm_Outer_CopperBottom" H 6100 7600 50  0001 C CNN
 F 3 "" H 6100 7600 50  0000 C CNN
 	1    5900 7600
@@
 F 0 "W2" V 6200 7650 50  0000 L CNN
 F 1 "FIDUCIAL2" V 6100 7900 50  0000 L CNN
-F 2 "Fiducials:Fiducial_1mm_Dia_2.54mm_Outer_CopperTop" H 6300 7600 50  0001 C CNN
+F 2 "GaudiLabsFootPrints:Fiducial_1mm_Dia_2.54mm_Outer_CopperBottom" H 6300 7600 50  0001 C CNN
 F 3 "" H 6300 7600 50  0000 C CNN
 	1    6100 7600
 	0    1    1    0
 $EndComp
-$Comp
-L OpenThereminV4-rescue:TEST_1P W3
-U 1 1 57DD73B6
-P 5950 1850
-F 0 "W3" V 5904 2037 50  0000 L CNN
-F 1 "TP1" V 5995 2037 50  0000 L CNN
-F 2 "Measurement_Points:Measurement_Point_Round-SMD-Pad_Small" H 6150 1850 50  0001 C CNN
-F 3 "" H 6150 1850 50  0000 C CNN
-	1    5950 1850
-	0    1    1    0
-$EndComp
-Wire Wire Line
-	5950 1850 5900 1850
-Connection ~ 5900 1850
-$Comp
-L OpenThereminV4-rescue:TEST_1P W4
-U 1 1 57DD87AC
-P 6000 5050
-F 0 "W4" V 5954 5237 50  0000 L CNN
-F 1 "TP2" V 6045 5237 50  0000 L CNN
-F 2 "Measurement_Points:Measurement_Point_Round-SMD-Pad_Small" H 6200 5050 50  0001 C CNN
-F 3 "" H 6200 5050 50  0000 C CNN
-	1    6000 5050
-	0    1    1    0
-$EndComp
-Connection ~ 6000 4550
 Wire Wire Line
 	2550 1100 2750 1100
@@
 Wire Wire Line
 	2550 2400 2550 2550
-Wire Wire Line
-	5900 1850 5900 1200
-Wire Wire Line
-	6000 4550 6000 5050
 Text Notes 5100 10500 0    60   ~ 0
 PITCH
@@
 	10350 3500 10200 3500
 Wire Wire Line
-	10200 3900 10850 3900
+	10200 3900 10600 3900
 Wire Wire Line
 	10850 3900 10850 3750
+Wire Wire Line
+	5900 1200 5900 2850
+$Comp
+L OpenThereminV4-rescue:CONN_01X01 P5
+U 1 1 6065CC3D
+P 6550 6050
+F 0 "P5" H 6469 5825 50  0000 C CNN
+F 1 "VCC" H 6850 6050 50  0000 C CNN
+F 2 "GaudiLabsFootPrints:SMD_Pinheader_1_OT_BLANK" H 6550 6050 50  0001 C CNN
+F 3 "" H 6550 6050 50  0000 C CNN
+	1    6550 6050
+	-1   0    0    1
+$EndComp
+Text GLabel 7100 6050 2    60   Input ~ 0
+RXD
+Wire Wire Line
+	7100 6050 6750 6050
+$Comp
+L OpenThereminV4-rescue:CONN_01X01 P7
+U 1 1 606C3E76
+P 10350 4250
+F 0 "P7" H 10269 4025 50  0000 C CNN
+F 1 "CV1" H 10650 4250 50  0000 C CNN
+F 2 "GaudiLabsFootPrints:SMD_Pinheader_1_OT_BLANK" H 10350 4250 50  0001 C CNN
+F 3 "" H 10350 4250 50  0000 C CNN
+	1    10350 4250
+	0    1    1    0
+$EndComp
+$Comp
+L OpenThereminV4-rescue:CONN_01X01 P15
+U 1 1 606C585A
+P 10600 4250
+F 0 "P15" H 10519 4025 50  0000 C CNN
+F 1 "CV2" H 10900 4250 50  0000 C CNN
+F 2 "GaudiLabsFootPrints:SMD_Pinheader_1_OT_BLANK" H 10600 4250 50  0001 C CNN
+F 3 "" H 10600 4250 50  0000 C CNN
+	1    10600 4250
+	0    1    1    0
+$EndComp
+Wire Wire Line
+	10350 3750 10350 4050
+Connection ~ 10350 3750
+Wire Wire Line
+	10600 3900 10600 4050
+Connection ~ 10600 3900
+Wire Wire Line
+	10600 3900 10850 3900
+$Comp
+L OpenThereminV4-rescue:CONN_01X01 P6
+U 1 1 6071B244
+P 10350 1850
+F 0 "P6" H 10269 1625 50  0000 C CNN
+F 1 "audio" H 10650 1850 50  0000 C CNN
+F 2 "GaudiLabsFootPrints:SMD_Pinheader_1_OT_BLANK" H 10350 1850 50  0001 C CNN
+F 3 "" H 10350 1850 50  0000 C CNN
+	1    10350 1850
+	0    1    1    0
+$EndComp
+Wire Wire Line
+	10350 1550 10350 1650
+Connection ~ 10350 1550
+$Comp
+L OpenThereminV4-rescue:CONN_01X01 P16
+U 1 1 6075D6EA
+P 10950 1850
+F 0 "P16" H 10869 1625 50  0000 C CNN
+F 1 "GND" H 11250 1850 50  0000 C CNN
+F 2 "GaudiLabsFootPrints:SMD_Pinheader_1_OT_BLANK" H 10950 1850 50  0001 C CNN
+F 3 "" H 10950 1850 50  0000 C CNN
+	1    10950 1850
+	0    1    1    0
+$EndComp
+Wire Wire Line
+	10950 1650 10700 1650
+Connection ~ 10700 1650
+Wire Wire Line
+	10700 1650 10700 2000
 $EndSCHEMATC
